Commit message: cometition ready

File: ros/src/robot_config/urdf/myrobot.urdf (robot description, URDF)
Before this commit: robot visual, 6 links, 5 joints
Links:
- added link camera_link; visual box size=0.035 0.035 0.013
Joints:
- added joint base_to_camera_link: type fixed, parent base_link, child camera_link, origin xyz=-0.4 -0.17 0.3 rpy=0 0 3.14159
- joint base_to_imu: origin xyz=0 0 0.4 rpy=3.1416 0 0 -> xyz=0 0 0.2 rpy=3.1416 0 0
